File: hardware/BME688_SPS3-.kicad_sch (KiCad schematic)
At the start: 6 parts, among them U401 BME688, U402 USBLC6-2P6

Commit message: BME/BDE pin update
Connections:
- net GND: now also U401.5 (SDO)
- net SCL: no longer U401.5 (SDO)
Changed lines of the file:
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@@
 		(color 0 0 0 0)
 	)
+	(junction
+		(at 121.92 119.38)
+		(diameter 0)
+		(color 0 0 0 0)
+	)
+	(wire
+		(pts
+			(xy 121.92 114.3) (xy 121.92 119.38)
+		)
+		(stroke
+			(width 0)
+			(type default)
+		)
+	)
 	(wire
 		(pts
@@
 		(pts
 			(xy 190.5 124.46) (xy 190.5 119.38)
+		)
+		(stroke
+			(width 0)
+			(type default)
+		)
+	)
+	(wire
+		(pts
+			(xy 118.11 114.3) (xy 121.92 114.3)
 		)
 		(stroke
@@
 	)
 	(hierarchical_label "SCL"
-		(shape bidirectional)
+		(shape input)
 		(at 87.63 114.3 180)
 		(effects
@@
 		(effects
 			(font
-				(size 1.27 1.27)
-			)
-			(justify left)
-		)
-	)
-	(hierarchical_label "SCL"
-		(shape input)
-		(at 118.11 114.3 0)
-		(effects
-			(font

Commit message: Merge .kicad_sch schematic updates from diego-pcb
Parts:
- added C401: 22uF, Capacitor_SMD:C_0805_2012Metric, symbol Device:C
- added L401: 4.7uH, Inductor_SMD:L_1210_3225Metric, symbol Device:L
- added U401: TPS613222ADBVR, pyronet_footprints:SOT95P280X145-5N, symbol pyronet_symbols:TPS613222ADBVR
- renumbered C401 to C402, C402 to C403, U401 to U402, U402 to U403
Connections:
- net +3.3V: now also L401.1
- net +5V: now also C401.2, U401.4 (VOUT)
- net GND: now also C401.1, U401.2 (GND)
- new net: L401.2, U401.1 (SW)
Other:
- moved on the sheet: C402, C403, D401, SPS30_Connector401, U402, U403

Commit message: 5VB PCB layout
Parts:
- added C401: 10uF, Capacitor_SMD:C_0402_1005Metric, symbol Device:C
- added C403, C404: 10uF, Capacitor_SMD:C_0603_1608Metric, symbol Device:C
- added C405: 2.2uF, Capacitor_SMD:C_0603_1608Metric, symbol Device:C
- added D401: D_Schottky, Diode_SMD:D_0805_2012Metric, symbol Device:D_Schottky
- added R401: R, Resistor_SMD:R_0402_1005Metric, symbol Device:R
- C402: renamed from C401; value 22uF -> 10uF; footprint Capacitor_SMD:C_0805_2012Metric -> Capacitor_SMD:C_0603_1608Metric
- L401: footprint Inductor_SMD:L_1210_3225Metric -> Inductor_SMD:L_1008_2520Metric
- renumbered C402 to C406, C403 to C407, D401 to D402
Connections:
- net +3.3V: now also C405.2
- net +5V: now also C401.1, C403.2, C404.2, D401.1 (K)
- net GND: now also C403.1, C404.1
- net at L401.2, U401.1 (SW): now also C405.1, D401.2 (A), R401.1
- new net: C401.2, R401.2
Other:
- moved on the sheet: C402, L401

Commit message: power layout WIP
Other:
- moved on the sheet: C401, C402, C403, C404, C405, D401, L401, R401, U401

Commit message: PCB update
Connections:
- net GND: now also C405.1
- net at D401.2 (A), L401.2, R401.1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: no longer C405.1
Other:
- moved on the sheet: C405
Changed lines of the file:
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@@
+	)
+	(junction
+		(at 201.93 119.38)
+		(diameter 0)
+		(color 0 0 0 0)
 	)
 	(junction
@@
 	)
 	(junction
-		(at 132.08 99.06)
+		(at 201.93 106.68)
 		(diameter 0)
 		(color 0 0 0 0)
 	)
 	(junction
-		(at 200.66 119.38)
+		(at 132.08 99.06)
 		(diameter 0)
 		(color 0 0 0 0)
@@
 	)
 	(junction
-		(at 200.66 106.68)
+		(at 252.73 118.11)
+		(diameter 0)
+		(color 0 0 0 0)
+	)
+	(junction
+		(at 243.84 106.68)
 		(diameter 0)
 		(color 0 0 0 0)
@@
 		(color 0 0 0 0)
 	)
-	(junction
-		(at 252.73 118.11)
-		(diameter 0)
-		(color 0 0 0 0)
-	)
-	(junction
-		(at 243.84 106.68)
-		(diameter 0)
-		(color 0 0 0 0)
-	)
 	(wire
 		(pts
@@
 	(wire
 		(pts
-			(xy 194.31 119.38) (xy 200.66 119.38)
-		)
-		(stroke
-			(width 0)
-			(type default)
-		)
-	)
-	(wire
-		(pts
 			(xy 77.47 118.11) (xy 77.47 119.38)
 		)
@@
 	(wire
 		(pts
-			(xy 200.66 119.38) (xy 200.66 128.27)
-		)
-		(stroke
-			(width 0)
-			(type default)
-		)
-	)
-	(wire
-		(pts
 			(xy 243.84 106.68) (xy 243.84 118.11)
 		)
@@
 	(wire
 		(pts
-			(xy 182.88 119.38) (xy 182.88 128.27)
-		)
-		(stroke
-			(width 0)
-			(type default)
-		)
-	)
-	(wire
-		(pts
 			(xy 243.84 125.73) (xy 252.73 125.73)
 		)
@@
 	(wire
 		(pts
+			(xy 201.93 106.68) (xy 219.71 106.68)
+		)
+		(stroke
+			(width 0)
+			(type default)
+		)
+	)
+	(wire
+		(pts
 			(xy 29.21 105.41) (xy 29.21 109.22)
 		)
@@
 	(wire
 		(pts
+			(xy 201.93 106.68) (xy 200.66 106.68)
+		)
+		(stroke
+			(width 0)
+			(type default)
+		)
+	)
+	(wire
+		(pts
 			(xy 132.08 116.84) (xy 134.62 116.84)
 		)
@@
 	(wire
 		(pts
-			(xy 182.88 128.27) (xy 186.69 128.27)
-		)
-		(stroke
-			(width 0)
-			(type default)
-		)
-	)
-	(wire
-		(pts
 			(xy 59.69 101.6) (xy 77.47 101.6)
 		)
@@
 	(wire
 		(pts
-			(xy 194.31 128.27) (xy 200.66 128.27)
-		)
-		(stroke
-			(width 0)
-			(type default)
-		)
-	)
-	(wire
-		(pts
 			(xy 132.08 99.06) (xy 132.08 106.68)
 		)
@@
 	(wire
 		(pts
-			(xy 200.66 119.38) (xy 201.93 119.38)
-		)
-		(stroke
-			(width 0)
-			(type default)
-		)
-	)
-	(wire
-		(pts
 			(xy 72.39 118.11) (xy 72.39 119.38)
 		)
@@
 	(wire
 		(pts
-			(xy 200.66 119.38) (xy 200.66 106.68)
-		)
-		(stroke
-			(width 0)
-			(type default)
-		)
-	)
-	(wire
-		(pts
-			(xy 200.66 106.68) (xy 219.71 106.68)
+			(xy 201.93 119.38) (xy 201.93 106.68)
+		)
+		(stroke
+			(width 0)
+			(type default)
+		)
+	)
+	(wire
+		(pts
+			(xy 194.31 119.38) (xy 201.93 119.38)
 		)
 		(stroke
@@
 	(symbol
 		(lib_id "Device:C")
-		(at 190.5 128.27 270)
+		(at 182.88 123.19 180)
 		(unit 1)
 		(exclude_from_sim no)
@@
 		(dnp no)
 		(property "Reference" "C405"
-			(at 188.468 121.92 90)
+			(at 189.738 125.476 0)
 			(effects
 				(font
@@
 		)
 		(property "Value" "2.2uF"
-			(at 188.214 123.952 90)
+			(at 190.754 122.682 0)
 			(effects
 				(font
@@
 		)
 		(property "Footprint" "Capacitor_SMD:C_0603_1608Metric"
-			(at 186.69 129.2352 0)
+			(at 181.9148 119.38 0)
 			(effects
 				(font
@@
 		)
 		(property "Datasheet" "~"
-			(at 190.5 128.27 0)
+			(at 182.88 123.19 0)
 			(effects
 				(font
@@
 		)
 		(property "Description" "Unpolarized capacitor"
-			(at 190.5 128.27 0)
+			(at 182.88 123.19 0)
 			(effects
 				(font
@@
 					(unit 1)
 				)
+			)
+		)
+	)
+	(symbol
+		(lib_id "power:GND")
+		(at 182.88 127 0)
+		(unit 1)
+		(exclude_from_sim no)
+		(in_bom yes)
+		(on_board yes)
+		(dnp no)
+		(fields_autoplaced yes)
+		(property "Reference" "#PWR0411"
+			(at 182.88 133.35 0)
+			(effects
+				(font
+					(size 1.27 1.27)
+				)
+				(hide yes)
+			)
+		)
+		(property "Value" "GND"
+			(at 182.88 132.08 0)
+			(effects
+				(font
+					(size 1.27 1.27)
+				)
+			)
+		)
+		(property "Footprint" ""
+			(at 182.88 127 0)
+			(effects
+				(font
+					(size 1.27 1.27)
+				)
+				(hide yes)
+			)
+		)
+		(property "Datasheet" ""
+			(at 182.88 127 0)
+			(effects
+				(font
+					(size 1.27 1.27)
+				)
+				(hide yes)
+			)
+		)
+		(property "Description" "Power symbol creates a global label with name \"GND\" , ground"
+			(at 182.88 127 0)
+			(effects
+				(font
+					(size 1.27 1.27)
+				)
+				(hide yes)
+			)
+		)
+		(pin "1"
+		)
+		(instances
+			(project "Senior_Design"
+				(path "/8f5928e8-0fc1-4443-a20f-3bfeb956761e/140ad835-eaa4-4a8c-a4e7-0525bbf22a2e"
+					(reference "#PWR0411")
+					(unit 1)
+				)

Commit message: PCB Layout update
Changed lines of the file:
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@@
 	(wire
 		(pts
-			(xy 200.66 106.68) (xy 200.66 95.25)
+			(xy 201.93 106.68) (xy 201.93 95.25)
 		)
 		(stroke
@@
 	(wire
 		(pts
-			(xy 200.66 95.25) (xy 209.55 95.25)
+			(xy 201.93 95.25) (xy 209.55 95.25)
 		)
 		(stroke
@@
 		)
 		(stroke
-			(width 0)
-			(type default)
-		)
-	)
-	(wire
-		(pts
-			(xy 201.93 106.68) (xy 200.66 106.68)
-		)
-		(stroke

Commit message: PCB Layout - Rev 1.0
Parts:
- renumbered C406 to C402, C407 to C403, C402 to C404, C403 to C405, C404 to C406, C405 to C407, D402 to D401, D401 to D402, U402 to U401, U403 to U402, U401 to U403
