File: hardware/BDE-MB1352P71UA32.kicad_sch (KiCad schematic)
At the start: 9 parts, among them J301 Conn_ARM_JTAG_SWD_10, SW301 SW_Push, U301 BDE-MB1352P71UA32

Commit message: BDE footprint/new 5V boost
Parts:
- U301: footprint pyronet_footprints:XCVR_BDE-MB1352P71UA32 -> pyronet_footprints:XCVR_BDE-MB1352P71UA32_1.03
Changed lines of the file:
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@@
 			)
 		)
-		(property "Footprint" "pyronet_footprints:XCVR_BDE-MB1352P71UA32"
+		(property "Footprint" "pyronet_footprints:XCVR_BDE-MB1352P71UA32_1.03"
 			(at 189.23 85.09 0)
 			(effects

Commit message: BME/BDE pin update
Connections:
- net BDE_DEBUG0: now also U301.36 (DIO_28); no longer U301.9 (DIO_7)
- net BDE_DEBUG1: now also U301.37 (DIO_29); no longer U301.16 (DIO_11)
Changed lines of the file:
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@@
+	)
+	(no_connect
+		(at 166.37 92.71)
 	)
 	(no_connect
@@
 	)
 	(no_connect
-		(at 212.09 97.79)
-	)
-	(no_connect
-		(at 212.09 95.25)
-	)
-	(no_connect
 		(at 166.37 87.63)
 	)
@@
 	(no_connect
 		(at 166.37 90.17)
+	)
+	(no_connect
+		(at 166.37 95.25)
 	)
 	(no_connect
@@
 	(hierarchical_label "BDE_DEBUG1"
 		(shape bidirectional)
-		(at 166.37 95.25 180)
-		(effects
-			(font
-				(size 1.27 1.27)
-			)
-			(justify right)
+		(at 212.09 97.79 0)
+		(effects
+			(font
+				(size 1.27 1.27)
+			)
+			(justify left)
 		)
 	)
@@
 	(hierarchical_label "BDE_DEBUG0"
 		(shape bidirectional)
-		(at 166.37 92.71 180)
-		(effects
-			(font
-				(size 1.27 1.27)
-			)
-			(justify right)
-		)
-	)
+		(at 212.09 95.25 0)
+		(effects
+			(font
+				(size 1.27 1.27)
+			)
+			(justify left)
+		)
+	)

Commit message: Merge .kicad_sch schematic updates from diego-pcb
Connections:
- net BDE_DEBUG0: now also U301.32 (DIO_24); no longer U301.36 (DIO_28)
- net BDE_DEBUG1: now also U301.31 (DIO_23); no longer U301.37 (DIO_29)
- net MCU_CTS_BDE_RTS: now also U301.33 (DIO_25); no longer U301.19 (DIO_14)
- net MCU_RTS_BDE_CTS: now also U301.34 (DIO_26); no longer U301.20 (DIO_15)
- net MCU_RX_BDE_TX: now also U301.35 (DIO_27); no longer U301.18 (DIO_13)
- net MCU_TX_BDE_RX: now also U301.36 (DIO_28); no longer U301.17 (DIO_12)
Changed lines of the file:
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@@
+	)
+	(no_connect
+		(at 212.09 97.79)
 	)
 	(no_connect
@@
 	)
 	(no_connect
-		(at 212.09 92.71)
-	)
-	(no_connect
 		(at 166.37 87.63)
 	)
 	(no_connect
+		(at 212.09 62.23)
+	)
+	(no_connect
 		(at 166.37 69.85)
 	)
 	(no_connect
-		(at 212.09 85.09)
-	)
-	(no_connect
 		(at 212.09 100.33)
 	)
@@
 	)
 	(no_connect
-		(at 212.09 90.17)
+		(at 166.37 100.33)
 	)
 	(no_connect
@@
 	)
 	(no_connect
+		(at 212.09 64.77)
+	)
+	(no_connect
+		(at 166.37 97.79)
+	)
+	(no_connect
 		(at 212.09 107.95)
 	)
 	(no_connect
-		(at 212.09 82.55)
-	)
-	(no_connect
-		(at 212.09 87.63)
-	)
-	(no_connect
 		(at 212.09 77.47)
 	)
@@
 	(wire
 		(pts
+			(xy 212.09 82.55) (xy 214.63 82.55)
+		)
+		(stroke
+			(width 0)
+			(type default)
+		)
+	)
+	(wire
+		(pts
 			(xy 140.97 62.23) (xy 166.37 62.23)
 		)
@@
 	(wire
 		(pts
+			(xy 212.09 85.09) (xy 214.63 85.09)
+		)
+		(stroke
+			(width 0)
+			(type default)
+		)
+	)
+	(wire
+		(pts
 			(xy 132.08 129.54) (xy 130.81 129.54)
 		)
@@
 	(wire
 		(pts
+			(xy 212.09 92.71) (xy 214.63 92.71)
+		)
+		(stroke
+			(width 0)
+			(type default)
+		)
+	)
+	(wire
+		(pts
 			(xy 232.41 45.72) (xy 232.41 46.99)
 		)
@@
 	(wire
 		(pts
+			(xy 212.09 95.25) (xy 214.63 95.25)
+		)
+		(stroke
+			(width 0)
+			(type default)
+		)
+	)
+	(wire
+		(pts
 			(xy 88.9 100.33) (xy 91.44 100.33)
 		)
@@
 	(wire
 		(pts
-			(xy 224.79 62.23) (xy 212.09 62.23)
+			(xy 212.09 87.63) (xy 214.63 87.63)
 		)
 		(stroke
@@
 	(wire
 		(pts
-			(xy 224.79 64.77) (xy 212.09 64.77)
-		)
-		(stroke
-			(width 0)
-			(type default)
-		)
-	)
-	(wire
-		(pts
 			(xy 213.36 113.03) (xy 212.09 113.03)
 		)
@@
 		(pts
 			(xy 76.2 116.84) (xy 76.2 118.11)
+		)
+		(stroke
+			(width 0)
+			(type default)
+		)
+	)
+	(wire
+		(pts
+			(xy 212.09 90.17) (xy 214.63 90.17)
 		)
 		(stroke
@@
 	(hierarchical_label "MCU_RTS_BDE_CTS"
 		(shape input)
-		(at 224.79 64.77 0)
+		(at 214.63 90.17 0)
 		(effects
 			(font
@@
 	(hierarchical_label "BDE_DEBUG1"
 		(shape bidirectional)
-		(at 212.09 97.79 0)
+		(at 214.63 82.55 0)
 		(effects
 			(font
@@
 	(hierarchical_label "MCU_CTS_BDE_RTS"
 		(shape output)
-		(at 224.79 62.23 0)
+		(at 214.63 87.63 0)
 		(effects
 			(font
@@
 	(hierarchical_label "MCU_TX_BDE_RX"
 		(shape input)
-		(at 166.37 97.79 180)
-		(effects
-			(font
-				(size 1.27 1.27)
-			)
-			(justify right)
+		(at 214.63 95.25 0)
+		(effects
+			(font
+				(size 1.27 1.27)
+			)
+			(justify left)
 		)
 	)
 	(hierarchical_label "MCU_RX_BDE_TX"
 		(shape output)
-		(at 166.37 100.33 180)
-		(effects
-			(font
-				(size 1.27 1.27)
-			)
-			(justify right)
+		(at 214.63 92.71 0)
+		(effects
+			(font
+				(size 1.27 1.27)
+			)
+			(justify left)
 		)
 	)
 	(hierarchical_label "BDE_DEBUG0"
 		(shape bidirectional)
-		(at 212.09 95.25 0)
-		(effects
-			(font
+		(at 214.63 85.09 0)
+		(effects
+			(font

Commit message: Rev 1.2 - debuggin pins added
Parts:
- added J302: Conn_01x05, Connector_PinHeader_2.54mm:PinHeader_1x05_P2.54mm_Vertical, symbol Connector_Generic:Conn_01x05
Connections:
- net BDE_DEBUG0: now also J302.5 (Pin_5)
- net MCU_CTS_BDE_RTS: now also J302.4 (Pin_4)
- net MCU_RTS_BDE_CTS: now also J302.3 (Pin_3)
- net MCU_RX_BDE_TX: now also J302.2 (Pin_2)
- net MCU_TX_BDE_RX: now also J302.1 (Pin_1)
Changed lines of the file:
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@@
+	)
+	(junction
+		(at 231.14 95.25)
+		(diameter 0)
+		(color 0 0 0 0)
+	)
+	(junction
+		(at 226.06 90.17)
+		(diameter 0)
+		(color 0 0 0 0)
+	)
+	(junction
+		(at 220.98 85.09)
+		(diameter 0)
+		(color 0 0 0 0)
+	)
+	(junction
+		(at 228.6 92.71)
+		(diameter 0)
+		(color 0 0 0 0)
 	)
 	(junction
@@
 	)
 	(junction
+		(at 223.52 87.63)
+		(diameter 0)
+		(color 0 0 0 0)
+	)
+	(junction
 		(at 219.71 57.15)
 		(diameter 0)
@@
 	(wire
 		(pts
+			(xy 223.52 87.63) (xy 223.52 99.06)
+		)
+		(stroke
+			(width 0)
+			(type default)
+		)
+	)
+	(wire
+		(pts
 			(xy 88.9 92.71) (xy 91.44 92.71)
 		)
@@
 	(wire
 		(pts
+			(xy 220.98 85.09) (xy 236.22 85.09)
+		)
+		(stroke
+			(width 0)
+			(type default)
+		)
+	)
+	(wire
+		(pts
 			(xy 132.08 124.46) (xy 130.81 124.46)
 		)
@@
 	(wire
 		(pts
+			(xy 226.06 90.17) (xy 226.06 99.06)
+		)
+		(stroke
+			(width 0)
+			(type default)
+		)
+	)
+	(wire
+		(pts
 			(xy 212.09 82.55) (xy 214.63 82.55)
 		)
@@
 	(wire
 		(pts
-			(xy 212.09 85.09) (xy 214.63 85.09)
+			(xy 212.09 85.09) (xy 220.98 85.09)
 		)
 		(stroke
@@
 	(wire
 		(pts
-			(xy 212.09 92.71) (xy 214.63 92.71)
+			(xy 212.09 92.71) (xy 228.6 92.71)
 		)
 		(stroke
@@
 	(wire
 		(pts
+			(xy 226.06 90.17) (xy 236.22 90.17)
+		)
+		(stroke
+			(width 0)
+			(type default)
+		)
+	)
+	(wire
+		(pts
 			(xy 213.36 50.8) (xy 213.36 57.15)
 		)
@@
 	(wire
 		(pts
+			(xy 231.14 95.25) (xy 231.14 99.06)
+		)
+		(stroke
+			(width 0)
+			(type default)
+		)
+	)
+	(wire
+		(pts
+			(xy 220.98 85.09) (xy 220.98 99.06)
+		)
+		(stroke
+			(width 0)
+			(type default)
+		)
+	)
+	(wire
+		(pts
 			(xy 232.41 46.99) (xy 232.41 48.26)
 		)
@@
 	(wire
 		(pts
-			(xy 212.09 95.25) (xy 214.63 95.25)
+			(xy 228.6 92.71) (xy 236.22 92.71)
+		)
+		(stroke
+			(width 0)
+			(type default)
+		)
+	)
+	(wire
+		(pts
+			(xy 212.09 95.25) (xy 231.14 95.25)
 		)
 		(stroke
@@
 	(wire
 		(pts
-			(xy 212.09 87.63) (xy 214.63 87.63)
+			(xy 212.09 87.63) (xy 223.52 87.63)
 		)
 		(stroke
@@
 	(wire
 		(pts
+			(xy 228.6 92.71) (xy 228.6 99.06)
+		)
+		(stroke
+			(width 0)
+			(type default)
+		)
+	)
+	(wire
+		(pts
 			(xy 213.36 113.03) (xy 212.09 113.03)
 		)
@@
 	(wire
 		(pts
-			(xy 212.09 90.17) (xy 214.63 90.17)
+			(xy 212.09 90.17) (xy 226.06 90.17)
 		)
 		(stroke
@@
 	(wire
 		(pts
+			(xy 231.14 95.25) (xy 236.22 95.25)
+		)
+		(stroke
+			(width 0)
+			(type default)
+		)
+	)
+	(wire
+		(pts
 			(xy 88.9 102.87) (xy 91.44 102.87)
+		)
+		(stroke
+			(width 0)
+			(type default)
+		)
+	)
+	(wire
+		(pts
+			(xy 223.52 87.63) (xy 236.22 87.63)
 		)
 		(stroke
@@
 	(hierarchical_label "MCU_RTS_BDE_CTS"
 		(shape input)
-		(at 214.63 90.17 0)
+		(at 236.22 90.17 0)
 		(effects
 			(font
@@
 	(hierarchical_label "MCU_CTS_BDE_RTS"
 		(shape output)
-		(at 214.63 87.63 0)
+		(at 236.22 87.63 0)
 		(effects
 			(font
@@
 	(hierarchical_label "MCU_TX_BDE_RX"
 		(shape input)
-		(at 214.63 95.25 0)
+		(at 236.22 95.25 0)
 		(effects
 			(font
@@
 	(hierarchical_label "MCU_RX_BDE_TX"
 		(shape output)
-		(at 214.63 92.71 0)
+		(at 236.22 92.71 0)
 		(effects
 			(font
@@
 	(hierarchical_label "BDE_DEBUG0"
 		(shape bidirectional)
-		(at 214.63 85.09 0)
+		(at 236.22 85.09 0)
 		(effects
 			(font
@@
 					(unit 1)
 				)
+			)
+		)
+	)
+	(symbol
+		(lib_id "Connector_Generic:Conn_01x05")
+		(at 226.06 104.14 270)
+		(unit 1)
+		(exclude_from_sim no)
+		(in_bom yes)
+		(on_board yes)
+		(dnp no)
+		(fields_autoplaced yes)
+		(property "Reference" "J302"
+			(at 226.06 107.95 90)
+			(effects
+				(font
+					(size 1.27 1.27)
+				)
+			)
+		)
+		(property "Value" "Conn_01x05"
+			(at 226.06 110.49 90)
+			(effects
+				(font
+					(size 1.27 1.27)
+				)
+			)
+		)
+		(property "Footprint" "Connector_PinHeader_2.54mm:PinHeader_1x05_P2.54mm_Vertical"
+			(at 226.06 104.14 0)
+			(effects
+				(font
+					(size 1.27 1.27)
+				)
+				(hide yes)
+			)
+		)
+		(property "Datasheet" "~"
+			(at 226.06 104.14 0)
+			(effects
+				(font
+					(size 1.27 1.27)
+				)
+				(hide yes)
+			)
+		)
+		(property "Description" "Generic connector, single row, 01x05, script generated (kicad-library-utils/schlib/autogen/connector/)"
+			(at 226.06 104.14 0)
+			(effects
+				(font
+					(size 1.27 1.27)
+				)
+				(hide yes)
+			)
+		)
+		(pin "2"
+		)
+		(pin "1"
+		)
+		(pin "3"
+		)
+		(pin "4"
+		)
+		(pin "5"
+		)
+		(instances
+			(project ""
+				(path "/8f5928e8-0fc1-4443-a20f-3bfeb956761e/dd2813e4-a810-44d7-8b7e-d46ce1c3fa30"
+					(reference "J302")
+					(unit 1)
+				)

Commit message: PCB cleanup
Changed lines of the file:
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@@
 	(wire
 		(pts
-			(xy 212.09 82.55) (xy 214.63 82.55)
+			(xy 212.09 82.55) (xy 236.22 82.55)
 		)
 		(stroke
@@
 	(hierarchical_label "BDE_DEBUG1"
 		(shape bidirectional)
-		(at 214.63 82.55 0)
-		(effects
-			(font
+		(at 236.22 82.55 0)
+		(effects
+			(font

Commit message: label cleanup
Parts:
- C303: value 0.1µF -> 0.1uF
- R301: value 100k -> 100K
- R302: value 10k -> 10K
Changed lines of the file:
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@@
 			)
 		)
-		(property "Value" "0.1µF"
+		(property "Value" "0.1uF"
 			(at 149.606 65.278 0)
 			(effects
@@
 			)
 		)
-		(property "Value" "100k"
+		(property "Value" "100K"
 			(at 143.002 56.642 0)
 			(effects
@@
 			)
 		)
-		(property "Value" "10k"
+		(property "Value" "10K"
 			(at 146.558 79.502 0)
 			(effects

Commit message: value update
Parts:
- C301: value 0.1uF -> 0R
- renumbered C302 to 0R
Changed lines of the file:
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@@
 			)
 		)
-		(property "Value" "0.1uF"
+		(property "Value" "0R"
 			(at 222.758 52.578 0)
 			(effects
@@
 		(dnp no)
 		(fields_autoplaced yes)
-		(property "Reference" "C302"
+		(property "Reference" "0R"
 			(at 236.22 50.7999 0)
 			(effects
@@
 			(project "Senior_Design"
 				(path "/8f5928e8-0fc1-4443-a20f-3bfeb956761e/dd2813e4-a810-44d7-8b7e-d46ce1c3fa30"
-					(reference "C302")
-					(unit 1)
-				)
+					(reference "0R")
+					(unit 1)
+				)
